File: PCB_Tester.kicad_pcb (KiCad board)
At the start: 2 copper layers, 100 x 100 mm, 61 parts, among them IC1 MCP4551-103E_MS, IC2 MCP4551-103E_MS, J1 Conn_01x14_Pin, J2 Conn_01x15_Pin, J3 Conn_01x04_Pin, U1 ULN2003A, U2 ULN2003A

Commit message: 1
Parts:
- removed IC1, IC2: MCP4551-103E_MS, Library:SOP65P490X110-8N
- removed R29, R30, R34, R35, R36, R37, R38, R39: R, Resistor_SMD:R_0805_2012Metric
- added C1: 1uF, Capacitor_SMD:C_0805_2012Metric, F.Cu at (169.2, 94.9)
- added C2: 1uF, Capacitor_SMD:C_0805_2012Metric, F.Cu at (171.7, 94.9)
- added C3: 1uF, Capacitor_SMD:C_0805_2012Metric, F.Cu at (169.1, 76.2)
- added C4: 1uF, Capacitor_SMD:C_0805_2012Metric, F.Cu at (171.6, 76.2)
- added C5: 1uF, Capacitor_SMD:C_0805_2012Metric, F.Cu at (168.2, 67.0)
- added C6: 1uF, Capacitor_SMD:C_0805_2012Metric, F.Cu at (170.7, 67.0)
- added C7: 1uF, Capacitor_SMD:C_0805_2012Metric, F.Cu at (169.1, 85.5)
- added C8: 1uF, Capacitor_SMD:C_0805_2012Metric, F.Cu at (171.6, 85.5)
- added Q1: AO3400A, Package_TO_SOT_SMD:SOT-23, F.Cu at (161.1, 83.9)
- added Q2: AO3400A, Package_TO_SOT_SMD:SOT-23, F.Cu at (161.0, 74.7)
- added R40: R, Resistor_SMD:R_0805_2012Metric, F.Cu at (165.6, 72.8)
- added R41: R, Resistor_SMD:R_0805_2012Metric, F.Cu at (166.6, 76.2)
- added R42: R, Resistor_SMD:R_0805_2012Metric, F.Cu at (170.1, 72.8)
- added R43: R, Resistor_SMD:R_0805_2012Metric, F.Cu at (164.7, 63.5)
- added R44: R, Resistor_SMD:R_0805_2012Metric, F.Cu at (165.7, 67.0)
- added R45: R, Resistor_SMD:R_0805_2012Metric, F.Cu at (169.2, 63.5)
- added R46: R, Resistor_SMD:R_0805_2012Metric, F.Cu at (165.6, 82.0)
- added R47: R, Resistor_SMD:R_0805_2012Metric, F.Cu at (166.6, 85.5)
- added R48: R, Resistor_SMD:R_0805_2012Metric, F.Cu at (170.1, 82.0)
- added R49: 10k, Resistor_SMD:R_0805_2012Metric, F.Cu at (157.6, 85.4)
- added R50: 10k, Resistor_SMD:R_0805_2012Metric, F.Cu at (157.6, 76.2)
- R31: value R -> 66k
- R32, R33: value R -> 10k
- moved J3 75.5 mm to (182.0, 54.5), turned to 0 degrees
- moved R33 13.6 mm to (170.2, 91.4), turned to 180 degrees
- moved R31 10.4 mm to (165.7, 91.4), turned to 180 degrees
- moved R32 9.31 mm to (166.7, 94.9), turned to -90 degrees
Connections:
- J2 pad 14: P0A_1 -> GND
- J2 pad 2: P0A_1 -> GND
- J3 pad 1: TC -> DPS
- J3 pad 2: CS -> BS
- J3 pad 3: BS -> FGS
- J3 pad 4: unconnected-(J3-Pin_4-Pad4) -> TC
- R31 pad 2: PWM -> TC_PWM
- R32 pad 2: P0A_1 -> GND
- U1 pad 8: P0A_1 -> unconnected-(U1-GND-Pad8)
- U2 pad 8: P0A_1 -> GND
- U3 pad 15: unconnected-(U3-PB7-Pad15) -> BS_PVM
- U3 pad 16: SCL_1 -> FGS_PVM
- U3 pad 17: SDA_1 -> TC_PWM
- U3 pad 19: P0A_1 -> GND
- U3 pad 37: PWM -> DPS_PVM
- U3 pad 39: P0A_1 -> GND
Routing:
- net GND: track 0.00 -> 40.8 mm
- net Net-(C1-Pad1): track 0.00 -> 7.94 mm
- net Net-(C5-Pad1): track 0.00 -> 7.92 mm
- net Net-(C7-Pad1): track 0.00 -> 7.73 mm
- net Net-(C3-Pad1): track 0.00 -> 7.57 mm
- net Net-(Q2-D): track 0.00 -> 4.06 mm
- net Net-(Q1-D): track 0.00 -> 4.00 mm
- net FGS: track 0.00 -> 2.84 mm
- net TC: track 0.00 -> 2.79 mm
- net DPS: track 0.00 -> 2.79 mm
- net BS: track 0.00 -> 2.74 mm
- net FGS_PVM: track 0.00 -> 2.71 mm
- net BS_PVM: track 0.00 -> 2.64 mm
